Commit message: created mapping launch file. parameters to be tuned and topics to be remapped.

File: catkin_ws/src/my_robot/urdf/my_robot.xacro (robot description, xacro)
@@ -189,5 +189,5 @@
     <material>Gazebo/Red</material>
   </gazebo>
-  <joint>
+  <joint name="camera_optical_joint" type="fixed">
     <origin xyz="0 0 0" rpy="-1.5707 0 -1.5707" />
     <parent link="camera" />
